File: Hardware/RegisterFile/regs.kicad_sch (KiCad schematic)
At the start: 17 parts, among them U1 74LS138

Commit message: RegisterFile Layout: Everything except the "spider" (routing the all 8 muxes each to all 8 registers might be non-trivial)
Parts:
- U1, UM0, UM1, UM2, UM3, UM4, UM5, UM6, UM7: footprint (none) -> 000custom:R-PDSO-G16
Changed lines of the file:
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@@
     (property "Reference" "UM4" (id 0) (at 226.06 67.31 0))
     (property "Value" "74151" (id 1) (at 236.22 67.31 0))
-    (property "Footprint" "" (id 2) (at 231.14 85.09 0)
+    (property "Footprint" "000custom:R-PDSO-G16" (id 2) (at 231.14 85.09 0)
       (effects (font (size 1.27 1.27)) hide)
     )
@@
     (property "Reference" "UM0" (id 0) (at 33.02 67.31 0))
     (property "Value" "74151" (id 1) (at 43.18 67.31 0))
-    (property "Footprint" "" (id 2) (at 38.1 85.09 0)
+    (property "Footprint" "000custom:R-PDSO-G16" (id 2) (at 38.1 85.09 0)
       (effects (font (size 1.27 1.27)) hide)
     )
@@
     (property "Reference" "UM6" (id 0) (at 322.58 67.31 0))
     (property "Value" "74151" (id 1) (at 332.74 67.31 0))
-    (property "Footprint" "" (id 2) (at 327.66 85.09 0)
+    (property "Footprint" "000custom:R-PDSO-G16" (id 2) (at 327.66 85.09 0)
       (effects (font (size 1.27 1.27)) hide)
     )
@@
     (property "Reference" "UM1" (id 0) (at 81.28 67.31 0))
     (property "Value" "74151" (id 1) (at 91.44 67.31 0))
-    (property "Footprint" "" (id 2) (at 86.36 85.09 0)
+    (property "Footprint" "000custom:R-PDSO-G16" (id 2) (at 86.36 85.09 0)
       (effects (font (size 1.27 1.27)) hide)
     )
@@
     (property "Reference" "U1" (id 0) (at 72.39 161.29 0))
     (property "Value" "74LS138" (id 1) (at 83.82 161.29 0))
-    (property "Footprint" "" (id 2) (at 78.74 170.18 0)
+    (property "Footprint" "000custom:R-PDSO-G16" (id 2) (at 78.74 170.18 0)
       (effects (font (size 1.27 1.27)) hide)
     )
@@
     (property "Reference" "UM5" (id 0) (at 274.32 67.31 0))
     (property "Value" "74151" (id 1) (at 284.48 67.31 0))
-    (property "Footprint" "" (id 2) (at 279.4 85.09 0)
+    (property "Footprint" "000custom:R-PDSO-G16" (id 2) (at 279.4 85.09 0)
       (effects (font (size 1.27 1.27)) hide)
     )
@@
     (property "Reference" "UM3" (id 0) (at 177.8 67.31 0))
     (property "Value" "74151" (id 1) (at 187.96 67.31 0))
-    (property "Footprint" "" (id 2) (at 182.88 85.09 0)
+    (property "Footprint" "000custom:R-PDSO-G16" (id 2) (at 182.88 85.09 0)
       (effects (font (size 1.27 1.27)) hide)
     )
@@
     (property "Reference" "UM2" (id 0) (at 129.54 67.31 0))
     (property "Value" "74151" (id 1) (at 139.7 67.31 0))
-    (property "Footprint" "" (id 2) (at 134.62 85.09 0)
+    (property "Footprint" "000custom:R-PDSO-G16" (id 2) (at 134.62 85.09 0)
       (effects (font (size 1.27 1.27)) hide)
     )
@@
     (property "Reference" "UM7" (id 0) (at 370.84 67.31 0))
     (property "Value" "74151" (id 1) (at 381 67.31 0))
-    (property "Footprint" "" (id 2) (at 375.92 85.09 0)
-      (effects (font (size 1.27 1.27)) hide)
-    )
+    (property "Footprint" "000custom:R-PDSO-G16" (id 2) (at 375.92 85.09 0)
+      (effects (font (size 1.27 1.27)) hide)
+    )
