File: Hardware/ALU/ALU.kicad_sch (KiCad schematic)
At the start: 34 parts

Commit message: ALU Schematic: A backup save before I realized Kicad doesn't seem to officially support hierarchical busses. Soon to replace all sheet busses with lines (I guess four lines isn't too many...)
Parts:
- added C10, C11, C12, C13, C14, C15, C9: .1uF, Capacitor_SMD:C_1206_3216Metric_Pad1.33x1.80mm_HandSolder, symbol Device:C
- C1, C2, C3, C4, C5, C6, C7, C8: renamed from C?; footprint (none) -> Capacitor_SMD:C_1206_3216Metric_Pad1.33x1.80mm_HandSolder
- J1, J2, J3: renamed from J?; footprint (none) -> Connector_PinHeader_2.54mm:PinHeader_2x08_P2.54mm_Horizontal
- U10: renamed from U?; value 74LS32 -> 74x32; footprint (none) -> 000custom:R-PDSO-G16
- U11, U9: renamed from U?; value 74LS08 -> 74x08; footprint (none) -> 000custom:R-PDSO-G16
- U12: renamed from U?; value 74LS377 -> 74x377; footprint (none) -> 000custom:R-PDSO-G16
- U13, U14: renamed from U?; value 74LS157 -> 74x157; footprint (none) -> 000custom:R-PDSO-G16
- U8: renamed from U?; value 74LS86 -> 74x86; footprint (none) -> 000custom:R-PDSO-G16
Connections:
- net CLK: now also J3.1 (Pin_1)
- net GND: now also J3.11 (Pin_11), J3.2 (Pin_2), J3.4 (Pin_4), J3.5 (Pin_5), J3.6 (Pin_6), J3.7 (Pin_7), J3.8 (Pin_8), J3.9 (Pin_9), U8.7 (GND), C10.2, C11.2, C12.2, C13.2, C14.2, C15.2, C9.2
- net IMMHIGH0: now also J2.5 (Pin_5)
- net IN_IMMEDIATE0: now also J2.9 (Pin_9)
- net IN_IMMEDIATE1: now also J2.11 (Pin_11)
- net IN_IMMEDIATE2: now also J2.13 (Pin_13)
- net IN_IMMEDIATE3: now also J2.15 (Pin_15)
- net IN_OPCODE0: now also J2.1 (Pin_1)
- net IN_OPCODE1: now also J2.3 (Pin_3)
- net IN_OPCODE3: now also J2.7 (Pin_7)
- net OUT_CARRY: now also J3.3 (Pin_3)
- net OUT_RX_ID0: now also J3.10 (Pin_10)
- net OUT_RX_ID1: now also J3.12 (Pin_12)
- net OUT_RX_ID2: now also J3.14 (Pin_14)
- net OUT_RX_ID3: now also J3.16 (Pin_16)
- net VCC: now also J3.13 (Pin_13), J3.15 (Pin_15), U8.14 (VCC), C10.1, C11.1, C12.1, C13.1, C14.1, C15.1, C9.1
- net IN_ACC0: now reaches J1.1 (Pin_1)
- net IN_REGDATA4: now reaches J1.10 (Pin_10)
- net IN_ACC5: now reaches J1.11 (Pin_11)
- net IN_REGDATA5: now reaches J1.12 (Pin_12)
- net IN_ACC6: now reaches J1.13 (Pin_13)
- net IN_REGDATA6: now reaches J1.14 (Pin_14)
- net IN_ACC7: now reaches J1.15 (Pin_15)
- net IN_REGDATA7: now reaches J1.16 (Pin_16)
- net IN_REGDATA0: now reaches J1.2 (Pin_2)
- net IN_ACC1: now reaches J1.3 (Pin_3)
- net IN_REGDATA1: now reaches J1.4 (Pin_4)
- net IN_ACC2: now reaches J1.5 (Pin_5)
- net IN_REGDATA2: now reaches J1.6 (Pin_6)
- net IN_ACC3: now reaches J1.7 (Pin_7)
- net IN_REGDATA3: now reaches J1.8 (Pin_8)
- net IN_ACC4: now reaches J1.9 (Pin_9)
Other:
- note added: "Register to write to (usually ACC)"
- note added: "TODO: - Make Footprints - Check All Pinouts - Layout - Traces - Order this and register file"
- note added: "The ALU operators Broken into two 4-bit ALUs"
- note added: "Unused"
- note added: "carry in on subtract"
- note removed: "The ALU logic"
- note removed: "sub"
- moved on the sheet: C1, C2, C3, C4, C5, C6, C7, C8, J1, J2, J3, U10B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

Commit message: ALU: About to increase modularity by moving opcode parsing out of ALU onto motherboard (would turn backplane into more of a motherboard).
Parts:
- C1, C10, C11, C12, C13, C14, C15, C2, C3, C4, C5, C6, C7, C8, C9: stock (none) -> 200
- J1, J2, J3: value Conn_02x08_Odd_Even -> connector_2x8; stock (none) -> 12
- U2MUX1: renamed from U13; footprint 000custom:R-PDSO-G16 -> 000custom:D_R-PDSO-G16; stock (none) -> 6; to buy (none) -> 20
- U2MUX2: renamed from U14; footprint 000custom:R-PDSO-G16 -> 000custom:D_R-PDSO-G16; stock (none) -> 6; to buy (none) -> 20
- UAND1: renamed from U9; footprint 000custom:R-PDSO-G16 -> 000custom:D_R-PDSO-G14; stock (none) -> 0; to buy (none) -> 20
- UAND2: renamed from U11; footprint 000custom:R-PDSO-G16 -> 000custom:D_R-PDSO-G14; stock (none) -> 0; to buy (none) -> 20
- UOR1: renamed from U10; footprint 000custom:R-PDSO-G16 -> 000custom:D_R-PDSO-G14; stock (none) -> 0; to buy (none) -> 20
- UREG1: renamed from U12; footprint 000custom:R-PDSO-G16 -> 000custom:ON-SOIC20-WB; stock (none) -> 32
- UXOR1: renamed from U8; footprint 000custom:R-PDSO-G16 -> 000custom:D_R-PDSO-G14; stock (none) -> 9; to buy (none) -> 20
Connections:
- net IMMHIGH0 renamed IN_OPCODE2
Other:
- removed sheet merge_result
- removed sheet split_acc
- removed sheet split_regdata
- sheet lower ports: added IN_ACC0, IN_ACC1, IN_ACC2, IN_ACC3, IN_IMMEDIATE0, IN_IMMEDIATE1, IN_IMMEDIATE2, IN_IMMEDIATE3, IN_REGDATA0, IN_REGDATA1, IN_REGDATA2, IN_REGDATA3, OPCODE0, OPCODE1, OPCODE2, OPCODE3, OUT_RESULT0, OUT_RESULT1, OUT_RESULT2, OUT_RESULT3; removed IN_ACC[3..0], IN_IMMEDIATE[3..0], IN_REGDATA[3..0], OPCODE[3..0], OUT_RESULT[3..0]
- sheet upper ports: added IN_ACC0, IN_ACC1, IN_ACC2, IN_ACC3, IN_IMMEDIATE0, IN_IMMEDIATE1, IN_IMMEDIATE2, IN_IMMEDIATE3, IN_REGDATA0, IN_REGDATA1, IN_REGDATA2, IN_REGDATA3, OPCODE0, OPCODE1, OPCODE2, OPCODE3, OUT_RESULT0, OUT_RESULT1, OUT_RESULT2, OUT_RESULT3; removed IN_ACC[3..0], IN_IMMEDIATE[3..0], IN_REGDATA[3..0], OPCODE[3..0], OUT_RESULT[3..0]
- note added: "Connectors"
- note added: "Decoupling Capacitors"
- note added: "TODO: - Layout - Traces - Order board"
- note added: "This gets: - High regdata - High acc - op2 for imm"
- note added: "True on SET, RB, WB"
- note removed: "TODO: - Make Footprints - Check All Pinouts - Layout - Traces - Order this and register file"
- moved on the sheet: C1, C10, C11, C12, C13, C14, C15, C2, C3, C4, C5, C6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

Commit message: ALU: Starting routing. Also passing this to kicad's github #collab
Parts:
- removed C10, C11, C12, C13, C14, C15, C7, C8, C9: .1uF, Capacitor_SMD:C_1206_3216Metric_Pad1.33x1.80mm_HandSolder, symbol Device:C
- removed unit 1 of UAND1
- removed unit 2 of UAND1
- removed unit 4 of UAND2
- removed unit 3 of UAND2
- removed unit 5 of UAND2
- removed UOR1: 74x32, 000custom:D_R-PDSO-G14, symbol 74xx:74LS32
- removed UXOR1: 74x86, 000custom:D_R-PDSO-G14, symbol 74xx:74LS86
- renumbered UAND2 to UAND1
Connections:
- net CHANGEOUT: now also J1.5 (Pin_5)
- net CLK: now also J1.15 (Pin_15); no longer J3.1 (Pin_1)
- net GND: now also J1.13 (Pin_13), J1.3 (Pin_3); no longer J3.2 (Pin_2), J3.4 (Pin_4), J3.5 (Pin_5), J3.6 (Pin_6), J3.7 (Pin_7), J3.8 (Pin_8)
- net IN_ACC0: now also J2.1 (Pin_1); no longer J1.1 (Pin_1)
- net IN_ACC1: now also J2.3 (Pin_3); no longer J1.3 (Pin_3)
- net IN_ACC2: now also J2.5 (Pin_5); no longer J1.5 (Pin_5)
- net IN_ACC3: now also J2.7 (Pin_7); no longer J1.7 (Pin_7)
- net IN_ACC4: now also J2.9 (Pin_9); no longer J1.9 (Pin_9)
- net IN_ACC5: now also J2.11 (Pin_11); no longer J1.11 (Pin_11)
- net IN_ACC6: now also J2.13 (Pin_13); no longer J1.13 (Pin_13)
- net IN_ACC7: now also J2.15 (Pin_15); no longer J1.15 (Pin_15)
- net IN_IMMEDIATE0: now also J1.2 (Pin_2); no longer J2.9 (Pin_9)
- net IN_IMMEDIATE1: now also J1.4 (Pin_4); no longer J2.11 (Pin_11)
- net IN_IMMEDIATE2: now also J1.6 (Pin_6); no longer J2.13 (Pin_13)
- net IN_IMMEDIATE3: now also J1.8 (Pin_8); no longer J2.15 (Pin_15)
- net IN_OPCODE0: now also J3.7 (Pin_7); no longer J2.1 (Pin_1)
- net IN_OPCODE1: now also J3.5 (Pin_5); no longer J2.3 (Pin_3)
- net IN_OPCODE2: now also J3.3 (Pin_3); no longer J2.5 (Pin_5)
- net IN_OPCODE3: now also J3.1 (Pin_1); no longer J2.7 (Pin_7)
- net IN_REGDATA0: now also J2.2 (Pin_2); no longer J1.2 (Pin_2)
- net IN_REGDATA1: now also J2.4 (Pin_4); no longer J1.4 (Pin_4)
- net IN_REGDATA2: now also J2.6 (Pin_6); no longer J1.6 (Pin_6)
- net IN_REGDATA3: now also J2.8 (Pin_8); no longer J1.8 (Pin_8)
- net IN_REGDATA4: now also J2.10 (Pin_10); no longer J1.10 (Pin_10)
- net IN_REGDATA5: now also J2.12 (Pin_12); no longer J1.12 (Pin_12)
- net IN_REGDATA6: now also J2.14 (Pin_14); no longer J1.14 (Pin_14)
- net IN_REGDATA7: now also J2.16 (Pin_16); no longer J1.16 (Pin_16)
- net OUT_CARRY: now also J1.11 (Pin_11); no longer J3.3 (Pin_3)
- net OUT_RESULT0: now also J3.16 (Pin_16); no longer J2.2 (Pin_2)
- net OUT_RESULT1: now also J3.14 (Pin_14); no longer J2.4 (Pin_4)
- net OUT_RESULT2: now also J3.12 (Pin_12); no longer J2.6 (Pin_6)
- net OUT_RESULT3: now also J3.10 (Pin_10); no longer J2.8 (Pin_8)
- net OUT_RESULT4: now also J3.8 (Pin_8); no longer J2.10 (Pin_10)
- net OUT_RESULT5: now also J3.6 (Pin_6); no longer J2.12 (Pin_12)
- net OUT_RESULT6: now also J3.4 (Pin_4); no longer J2.14 (Pin_14)
- net OUT_RESULT7: now also J3.2 (Pin_2); no longer J2.16 (Pin_16)
- net OUT_RX_ID0: now also J1.10 (Pin_10); no longer J3.10 (Pin_10)
- net OUT_RX_ID1: now also J1.12 (Pin_12); no longer J3.12 (Pin_12)
- net OUT_RX_ID2: now also J1.14 (Pin_14); no longer J3.14 (Pin_14)
- net OUT_RX_ID3: now also J1.16 (Pin_16); no longer J3.16 (Pin_16)
- net SWAP_NIBBLES: now also J1.9 (Pin_9)
- net VCC: now also J1.1 (Pin_1)
- net ~{CARRY_WE}: now reaches UREG1.1 (~{E})
- net ~{CARRY_WE}: now also J1.7 (Pin_7)
- no-connect marks 10 -> 7
Other:
- note added: "Power comes from the connectors"
- note removed: "TODO: - Layout - Traces - Order board"
- note removed: "This gets: - High regdata - High acc - op2 for imm"
- note removed: "Unused"
- note removed: "only WE on add/sub"
- moved on the sheet: C1, C2, C3, C4, C5, C6, J1, J2, J3, UAND1A, UAND1B, UAND1C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
