File: Hardware/Motherboard/Motherboard.kicad_sch (KiCad schematic)
At the start: 54 parts, among them J1 PowerBarrel, SW1 Reset, U1 U04, U2MUX1 74x157, U2MUX2 74x157, U2MUX3 74x157, U2MUX4 74x157, U5 74x138, Y1 Crystal

Commit message: Switch the compiler to Java
Parts:
- added U?: 74x00, symbol 74xx:74LS00
Connections:
- net CEP is gone; now on net VCC: UR1.7 (CEP), UR2.7 (CEP), UR3.7 (CEP), UR4.7 (CEP)
- net ~{IS_SKIP}: now also U?.10
- net ~{MEM_WE}: now also U?.8; no longer UNAND1.8, UXOR1.5
- net ~{INST_MEM_WE}: now reaches UNOT1.5
- net ~{INST_MEM_WE}: now also UNAND1.8, UXOR1.5
- net INST_MEM_WE: now reaches UNOT1.6
- net INST_MEM_WE: now also U?.9
- net IS_JUMP renamed INST_JUMP
- net IS_SKIP renamed INST_SKIP
Other:
- sheet Daughter Boards ports: added OUT_RX_ID; removed none
- note added: "Skip has to do the following to the next instruction: ? Don't change carry register ? Don't change register file ? Don't write to memory"
- moved on the sheet: UNOT1C, UOR1D, UXOR1B, UXOR1C, UXOR1D

Commit message: Motherboard Schematic Major Updates:  - Skip implemented  - Memory WB implemented Also, the JavaAssembler was somewhat updated but isn't done yet.
Parts:
- removed D1: 5V Zener, symbol Device:D_Zener
- removed U?: 74x00, symbol 74xx:74LS00
- removed UCMP1: 74x684, 000custom:SOIC20_TI_DW0020A, symbol 74xx_IEEE:74LS684
- added JALU1, JALU2, JALU3, JMEM_A1, JMEM_A2, JMEM_B1, JMEM_B2, JMEM_C1, JMEM_C2, JMEM_D1, JMEM_D2, JREGHIGH1, JREGHIGH2, JREGHIGH3, JREGHIGH4, JREGLOW1, JREGLOW2: Conn2x8, Connector_PinSocket_2.54mm:PinSocket_2x08_P2.54mm_Vertical, symbol Connector_Generic:Conn_02x08_Odd_Even
- added JDBG1: Conn_02x11, Connector_PinHeader_2.54mm:PinHeader_2x11_P2.54mm_Vertical, symbol Connector_Generic:Conn_02x11_Odd_Even
- added TPROM15: ROMADDR15, symbol Connector:TestPoint
- added U2: AT28HC256, aFootprint:AMPHENOL_54020-32030LF, symbol 0MySym:AT28HC256
- added U3: APX823-46W5G-7, 000custom:SOT25, symbol 0MySym:APX823
- added U4: 74HCS244, 000custom:SOIC20_TI_DW0020A, symbol 74xx:74AHCT244
- added UOR2: 74x32, 000custom:D_R-PDSO-G14, symbol 74xx:74LS32
- added UREG1: 74x377, 000custom:ON-SOIC20-WB, symbol 74xx:74LS377
- R1: renamed from R2; footprint Resistor_SMD:R_1206_3216Metric_Pad1.30x1.75mm_HandSolder -> Resistor_SMD:R_0603_1608Metric_Pad0.98x0.95mm_HandSolder
- R2: renamed from R3; value 5k -> ~5k
- U1: value U04 -> INV_U04
- UDEMUX1: renamed from U5; footprint 000custom:R-PDSO-G16 -> 000custom:D_R-PDSO-G16
- renumbered C2 to C1, C8 to C10, C9 to C11, C10 to C12, C11 to C13, C12 to C14, C13 to C15, C14 to C16, C15 to C17, C16 to C18, C17 to C19, C3 to C2, C18 to C20, C19 to C21, C20 to C22, C21 to C23, C22 to C24, C23 to C25, C24 to C26, C25 to C27, C26 to C28, C4 to C3, C27 to C4, C1 to C6, C6 to C7, C28 to C8, C7 to C9, UNOT2 to UNOT1, UNOT1 to UNOT2, UCONDMUX1 to UOCTMUX1
Connections:
- net CLK_WB is gone; now on net CLK: UR1.2 (CP), UR2.2 (CP), UR3.2 (CP), UR4.2 (CP)
- net IN_IMMEDIATE3 is gone; now on net IMM3: U2MUX1.1 (S), U2MUX2.1 (S)
- net MEM_DATA7 is gone; now on net GND: U2MUX4.14 (I0d)
- net ALU_RESULT0: now also JALU3.8 (Pin_8)
- net ALU_RESULT1: now also JALU3.7 (Pin_7)
- net ALU_RESULT2: now also JALU3.6 (Pin_6)
- net ALU_RESULT3: now also JALU3.5 (Pin_5)
- net ALU_RESULT4: now also JALU3.4 (Pin_4)
- net ALU_RESULT5: now also JALU3.3 (Pin_3)
- net ALU_RESULT6: now also JALU3.2 (Pin_2)
- net ALU_RESULT7: now also JALU3.1 (Pin_1)
- net CARRY: now also JALU1.11 (Pin_11), JDBG1.13 (Pin_13)
- net CLK: now also JALU1.15 (Pin_15), JDBG1.12 (Pin_12), JMEM_A2.4 (Pin_4), JMEM_B2.4 (Pin_4), JMEM_C2.4 (Pin_4), JMEM_D2.4 (Pin_4), JREGHIGH1.5 (Pin_5), JREGLOW1.5 (Pin_5), UREG1.11 (CP)
- net DATAIN0: now also JREGHIGH4.7 (Pin_7), JREGLOW2.7 (Pin_7)
- net DATAIN1: now also JREGHIGH4.8 (Pin_8), JREGLOW2.8 (Pin_8)
- net DATAIN2: now also JREGHIGH4.5 (Pin_5), JREGLOW2.5 (Pin_5)
- net DATAIN3: now also JREGHIGH4.6 (Pin_6), JREGLOW2.6 (Pin_6)
- net DATAIN4: now also JREGHIGH4.3 (Pin_3), JREGLOW2.3 (Pin_3)
- net DATAIN5: now also JREGHIGH4.4 (Pin_4), JREGLOW2.4 (Pin_4)
- net DATAIN6: now also JREGHIGH4.1 (Pin_1), JREGLOW2.1 (Pin_1)
- net DATAIN7: now also JREGHIGH4.2 (Pin_2), JREGLOW2.2 (Pin_2)
- net DATAOUT_HIGH0: now also JREGHIGH4.15 (Pin_15)
- net DATAOUT_HIGH1: now also JREGHIGH4.16 (Pin_16)
- net DATAOUT_HIGH2: now also JREGHIGH4.13 (Pin_13)
- net DATAOUT_HIGH3: now also JREGHIGH4.14 (Pin_14)
- net DATAOUT_HIGH4: now also JREGHIGH4.11 (Pin_11)
- net DATAOUT_HIGH5: now also JREGHIGH4.12 (Pin_12)
- net DATAOUT_HIGH6: now also JREGHIGH4.9 (Pin_9)
- net DATAOUT_HIGH7: now also JREGHIGH4.10 (Pin_10)
- net DATAOUT_LOW0: now also JREGLOW2.15 (Pin_15)
- net DATAOUT_LOW1: now also JREGLOW2.16 (Pin_16)
- net DATAOUT_LOW2: now also JREGLOW2.13 (Pin_13)
- net DATAOUT_LOW3: now also JREGLOW2.14 (Pin_14)
- net DATAOUT_LOW4: now also JREGLOW2.11 (Pin_11)
- net DATAOUT_LOW5: now also JREGLOW2.12 (Pin_12)
- net DATAOUT_LOW6: now also JREGLOW2.9 (Pin_9)
- net DATAOUT_LOW7: now also JREGLOW2.10 (Pin_10)
- net GND: now also SW1.1, UNOT2.1, JALU2.11 (Pin_11), JALU3.13 (Pin_13), JDBG1.1 (Pin_1), JDBG1.14 (Pin_14), JMEM_A2.14 (Pin_14), JMEM_A2.15 (Pin_15), JMEM_A2.16 (Pin_16), JMEM_A2.2 (Pin_2), JMEM_B2.14 (Pin_14), JMEM_B2.15 (Pin_15), JMEM_B2.16 (Pin_16), JMEM_B2.2 (Pin_2), JMEM_C2.14 (Pin_14), JMEM_C2.15 (Pin_15), JMEM_C2.16 (Pin_16), JMEM_C2.2 (Pin_2), JMEM_D2.14 (Pin_14), JMEM_D2.15 (Pin_15), JMEM_D2.16 (Pin_16), JMEM_D2.2 (Pin_2), JREGHIGH1.1 (Pin_1), JREGHIGH1.15 (Pin_15), JREGHIGH1.2 (Pin_2), JREGHIGH1.4 (Pin_4), JREGHIGH1.9 (Pin_9), JREGLOW1.1 (Pin_1), JREGLOW1.15 (Pin_15), JREGLOW1.2 (Pin_2), JREGLOW1.4 (Pin_4), U2.16 (GND), U2.23 (~{CE}), U2.25 (~{OE}), U3.2 (GND), U4.10 (GND), U4.9 (2Y3), UOR2.7 (GND), UREG1.1 (~{E}), UREG1.10 (GND), UREG1.13 (D4), UREG1.14 (D5), UREG1.17 (D6), UREG1.18 (D7), UREG1.4 (D1), UREG1.7 (D2), UREG1.8 (D3)
- net IMM0: now also JALU1.16 (Pin_16), JDBG1.19 (Pin_19), JREGHIGH1.16 (Pin_16), JREGLOW1.16 (Pin_16), U2.19 (IO4)
- net IMM1: now also JALU1.14 (Pin_14), JDBG1.20 (Pin_20), JREGHIGH1.14 (Pin_14), JREGLOW1.14 (Pin_14), U2.20 (IO5)
- net IMM2: now also JALU1.12 (Pin_12), JDBG1.21 (Pin_21), JREGHIGH1.12 (Pin_12), JREGLOW1.12 (Pin_12), U2.21 (IO6)
- net IMM3: now also JALU1.10 (Pin_10), JDBG1.22 (Pin_22), U2.22 (IO7)
- net INST_JUMP: now also UNOT2.8; no longer UNOT1.2
- net IN_R1: now also JALU3.12 (Pin_12), JDBG1.16 (Pin_16), U2.14 (IO1)
- net IN_R2: now also UXOR1.8, JALU3.14 (Pin_14); no longer UOR1.6
- net IN_R3: now also UXOR1.11, JALU3.16 (Pin_16); no longer UOR1.8
- net MEM_DATA0: now also JMEM_A2.7 (Pin_7), JMEM_B2.7 (Pin_7), JMEM_C2.7 (Pin_7), JMEM_D2.7 (Pin_7), U4.18 (1Y0)
- net MEM_DATA1: now also JMEM_A2.8 (Pin_8), JMEM_B2.8 (Pin_8), JMEM_C2.8 (Pin_8), JMEM_D2.8 (Pin_8), U4.16 (1Y1)
- net MEM_DATA2: now also JMEM_A2.9 (Pin_9), JMEM_B2.9 (Pin_9), JMEM_C2.9 (Pin_9), JMEM_D2.9 (Pin_9), U4.14 (1Y2)
- net MEM_DATA3: now also JMEM_A2.10 (Pin_10), JMEM_B2.10 (Pin_10), JMEM_C2.10 (Pin_10), JMEM_D2.10 (Pin_10), U4.12 (1Y3)
- net MEM_DATA4: now also JMEM_A2.11 (Pin_11), JMEM_B2.11 (Pin_11), JMEM_C2.11 (Pin_11), JMEM_D2.11 (Pin_11), U4.3 (2Y0)
- net MEM_DATA5: now also JMEM_A2.12 (Pin_12), JMEM_B2.12 (Pin_12), JMEM_C2.12 (Pin_12), JMEM_D2.12 (Pin_12), U4.5 (2Y1)
- net MEM_DATA6: now also JMEM_A2.13 (Pin_13), JMEM_B2.13 (Pin_13), JMEM_C2.13 (Pin_13), JMEM_D2.13 (Pin_13), U4.7 (2Y2)
- net NEWCOND: now also UOCTMUX1.13 (I6), JDBG1.11 (Pin_11); no longer UOCTMUX1.3 (I1)
- net OPB_IS_IMM: now also JALU2.13 (Pin_13), JDBG1.15 (Pin_15), U2.13 (IO0)
- net OPCODE2: now also UXOR1.10, JDBG1.17 (Pin_17), U2.15 (IO2), UOR2.12; no longer UOR1.1, UOR1.5
- net OPCODE3: now also UXOR1.13, JDBG1.18 (Pin_18), U2.18 (IO3), UOR2.13; no longer UOR1.10, UOR1.2
- net OSC_OUT: now also UNOT1.1; no longer UNOT2.9
- net RCS0: now also UOCTMUX1.3 (I1), UOR1.1, JREGHIGH2.7 (Pin_7); no longer UOCTMUX1.2 (I2)
- net RCS1: now also UOR1.2, JREGHIGH2.8 (Pin_8)
- net RCS2: now also UOR1.4, JREGHIGH2.5 (Pin_5)
- net RCS3: now also UOR1.5, JREGHIGH2.6 (Pin_6)
- net RCS4: now also UOR1.9, JREGHIGH2.3 (Pin_3)
- net RCS5: now also UOR1.10, JREGHIGH2.4 (Pin_4)
- net RCS6: now also UOR1.12, JREGHIGH2.1 (Pin_1)
- net RCS7: now also UOCTMUX1.2 (I2), UOR1.13, JREGHIGH2.2 (Pin_2); no longer UOCTMUX1.1 (I3)
- net ROMADDR0: now also U2.11 (A0)
- net ROMADDR1: now also U2.10 (A1)
- net ROMADDR10: now also U2.24 (A10)
- net ROMADDR11: now also U2.27 (A11)
- net ROMADDR12: now also U2.3 (A12)
- net ROMADDR13: now also U2.30 (A13)
- net ROMADDR14: now also U2.2 (A14)
- net ROMADDR15: now also TPROM15.1
- net ROMADDR2: now also U2.9 (A2)
- net ROMADDR3: now also U2.8 (A3)
- net ROMADDR4: now also U2.7 (A4)
- net ROMADDR5: now also U2.6 (A5)
- net ROMADDR6: now also U2.5 (A6)
- net ROMADDR7: now also U2.4 (A7)
- net ROMADDR8: now also U2.29 (A8)
- net ROMADDR9: now also U2.28 (A9)
- net SWAP_NIBBLES: now also JALU3.11 (Pin_11)
- net VCC: now also JALU2.9 (Pin_9), JALU3.15 (Pin_15), JDBG1.2 (Pin_2), JMEM_A2.1 (Pin_1), JMEM_B2.1 (Pin_1), JMEM_C2.1 (Pin_1), JMEM_D2.1 (Pin_1), JREGHIGH1.13 (Pin_13), JREGHIGH1.3 (Pin_3), JREGLOW1.13 (Pin_13), JREGLOW1.3 (Pin_3), JREGLOW1.7 (Pin_7), U2.31 (~{WE}), U2.32 (VCC), U3.5 (VCC), U4.20 (VCC), UOR2.14 (VCC), UREG1.20 (VCC); no longer UDEMUX1.6 (G1)
- net ~{D0}: now also UXOR1.12, UXOR1.9; no longer UNOT2.1
- net ~{IS_SKIP}: now also UREG1.3 (D0)
- net ~{L}: now also UNAND1.2, JALU3.9 (Pin_9), UOR2.11; no longer UOR1.3
- net ~{REG_WE}: now also JREGHIGH1.11 (Pin_11), JREGLOW1.11 (Pin_11)
- net ~{RST}: now also JMEM_A2.3 (Pin_3), JMEM_B2.3 (Pin_3), JMEM_C2.3 (Pin_3), JMEM_D2.3 (Pin_3), U3.1 (~{RESET})
- net at JP1.1 (A): now also UNOT1.2; no longer UNOT2.8
- net at UNAND2.8: now also UNOT2.9; no longer UNOT1.1
- net at UOR1.11: now also UOR2.5
- net at SW1.2: now also U3.3 (~{MR})
- removed net D0: UNOT2.2, UOR1.4, UOR1.9
- net D1 renamed IN_R0
- net IN_R0: now also JALU3.10 (Pin_10)
- net D4 renamed IMM_MSB
- net IMM_MSB: now also JALU2.15 (Pin_15)
- net D5 renamed OUT_RX_ID
- net OUT_RX_ID: now also JALU1.13 (Pin_13)
- net INST_MEM_WE renamed ~{CARRY_WE}
- net ~{CARRY_WE}: now also JALU1.9 (Pin_9)
- net OUT_REGDATA0 renamed REGDATA0
- net REGDATA0: now also JALU1.7 (Pin_7), U4.2 (1A0)
- net OUT_REGDATA1 renamed REGDATA1
- net REGDATA1: now also JALU1.5 (Pin_5), U4.4 (1A1)
- net OUT_REGDATA2 renamed REGDATA2
- net REGDATA2: now also JALU1.3 (Pin_3), U4.6 (1A2)
- net OUT_REGDATA3 renamed REGDATA3
- net REGDATA3: now also JALU1.1 (Pin_1), U4.8 (1A3)
- net OUT_REGDATA4 renamed REGDATA4
- net REGDATA4: now also JALU1.8 (Pin_8), U4.17 (2A0)
- net OUT_REGDATA5 renamed REGDATA5
- net REGDATA5: now also JALU1.6 (Pin_6), U4.15 (2A1)
- net OUT_REGDATA6 renamed REGDATA6
- net REGDATA6: now also JALU1.4 (Pin_4), U4.13 (2A2)
- net OUT_REGDATA7 renamed REGDATA7
- net REGDATA7: now also JALU1.2 (Pin_2), U4.11 (2A3)
- net OVERFLOW: no longer names the net of UR4.15 (TC)
- net REGMEM0 renamed MEM_ADDR0
- net MEM_ADDR0: now also JMEM_A1.1 (Pin_1), JMEM_B1.1 (Pin_1), JMEM_C1.1 (Pin_1), JMEM_D1.1 (Pin_1), JREGHIGH3.7 (Pin_7)
- net REGMEM1 renamed MEM_ADDR1
- net MEM_ADDR1: now also JMEM_A1.2 (Pin_2), JMEM_B1.2 (Pin_2), JMEM_C1.2 (Pin_2), JMEM_D1.2 (Pin_2), JREGHIGH3.8 (Pin_8)
- net REGMEM10 renamed MEM_ADDR10
- net MEM_ADDR10: now also JMEM_A1.11 (Pin_11), JMEM_B1.11 (Pin_11), JMEM_C1.11 (Pin_11), JMEM_D1.11 (Pin_11), JREGHIGH3.13 (Pin_13)
- net REGMEM11 renamed MEM_ADDR11
- net MEM_ADDR11: now also JMEM_A1.12 (Pin_12), JMEM_B1.12 (Pin_12), JMEM_C1.12 (Pin_12), JMEM_D1.12 (Pin_12), JREGHIGH3.14 (Pin_14)
- net REGMEM12 renamed MEM_ADDR12
- net MEM_ADDR12: now also JMEM_A1.13 (Pin_13), JMEM_B1.13 (Pin_13), JMEM_C1.13 (Pin_13), JMEM_D1.13 (Pin_13), JREGHIGH3.11 (Pin_11)
- net REGMEM13 renamed MEM_ADDR13
- net MEM_ADDR13: now also JMEM_A1.14 (Pin_14), JMEM_B1.14 (Pin_14), JMEM_C1.14 (Pin_14), JMEM_D1.14 (Pin_14), JREGHIGH3.12 (Pin_12)
- net REGMEM14 renamed MEM_ADDR14
- net MEM_ADDR14: now also JMEM_A1.15 (Pin_15), JMEM_B1.15 (Pin_15), JMEM_C1.15 (Pin_15), JMEM_D1.15 (Pin_15), JREGHIGH3.9 (Pin_9)
- net REGMEM15 renamed MEM_ADDR15
- net MEM_ADDR15: now also JMEM_A1.16 (Pin_16), JMEM_B1.16 (Pin_16), JMEM_C1.16 (Pin_16), JMEM_D1.16 (Pin_16), JREGHIGH3.10 (Pin_10)
- net REGMEM2 renamed MEM_ADDR2
- net MEM_ADDR2: now also JMEM_A1.3 (Pin_3), JMEM_B1.3 (Pin_3), JMEM_C1.3 (Pin_3), JMEM_D1.3 (Pin_3), JREGHIGH3.5 (Pin_5)
- net REGMEM3 renamed MEM_ADDR3
- net MEM_ADDR3: now also JMEM_A1.4 (Pin_4), JMEM_B1.4 (Pin_4), JMEM_C1.4 (Pin_4), JMEM_D1.4 (Pin_4), JREGHIGH3.6 (Pin_6)
- net REGMEM4 renamed MEM_ADDR4
- net MEM_ADDR4: now also JMEM_A1.5 (Pin_5), JMEM_B1.5 (Pin_5), JMEM_C1.5 (Pin_5), JMEM_D1.5 (Pin_5), JREGHIGH3.3 (Pin_3)
- net REGMEM5 renamed MEM_ADDR5
- net MEM_ADDR5: now also JMEM_A1.6 (Pin_6), JMEM_B1.6 (Pin_6), JMEM_C1.6 (Pin_6), JMEM_D1.6 (Pin_6), JREGHIGH3.4 (Pin_4)
- net REGMEM6 renamed MEM_ADDR6
- net MEM_ADDR6: now also JMEM_A1.7 (Pin_7), JMEM_B1.7 (Pin_7), JMEM_C1.7 (Pin_7), JMEM_D1.7 (Pin_7), JREGHIGH3.1 (Pin_1)
- net REGMEM7 renamed MEM_ADDR7
- net MEM_ADDR7: now also JMEM_A1.8 (Pin_8), JMEM_B1.8 (Pin_8), JMEM_C1.8 (Pin_8), JMEM_D1.8 (Pin_8), JREGHIGH3.2 (Pin_2)
- net REGMEM8 renamed MEM_ADDR8
- net MEM_ADDR8: now also JMEM_A1.9 (Pin_9), JMEM_B1.9 (Pin_9), JMEM_C1.9 (Pin_9), JMEM_D1.9 (Pin_9), JREGHIGH3.15 (Pin_15)
- net REGMEM9 renamed MEM_ADDR9
- net MEM_ADDR9: now also JMEM_A1.10 (Pin_10), JMEM_B1.10 (Pin_10), JMEM_C1.10 (Pin_10), JMEM_D1.10 (Pin_10), JREGHIGH3.16 (Pin_16)
- net cmpeq renamed IN_ACC7
- net IN_ACC7: now also JALU2.1 (Pin_1), JDBG1.10 (Pin_10), JREGHIGH2.10 (Pin_10); no longer UNAND1.1
- net cmpgt renamed IN_ACC0
- net IN_ACC0: now also JALU2.8 (Pin_8), JDBG1.3 (Pin_3), JREGHIGH2.15 (Pin_15); no longer UNAND1.2
- net cmplt: no longer names the net of UNAND1.3
- net cmplt: now also UNOT1.5; no longer UOCTMUX1.13 (I6)
- net ~{INST_MEM_WE} renamed ~{INST_WB}
- net ~{INST_WB}: now also JMEM_A2.6 (Pin_6), JMEM_B2.6 (Pin_6), JMEM_C2.6 (Pin_6), JMEM_D2.6 (Pin_6), U4.1 (1OE), U4.19 (2OE); no longer UNOT1.5
- net ~{MEMORY_READ} renamed ~{MEM_OE}
- net ~{MEM_OE}: now also JMEM_A2.5 (Pin_5), JMEM_B2.5 (Pin_5), JMEM_C2.5 (Pin_5), JMEM_D2.5 (Pin_5)
- new net: UOR1.6, UOR2.2
- new net: UOR1.3, UOR2.1
- new net: UOCTMUX1.1 (I3), UOR2.8
- new net: UOR2.10, UOR2.6
- new net: UOR2.3, UOR2.9
- new net: UOR1.8, UOR2.4
- new net IN_ACC1: JALU2.6 (Pin_6), JDBG1.4 (Pin_4), JREGHIGH2.16 (Pin_16)
- new net IN_ACC2: JALU2.4 (Pin_4), JDBG1.5 (Pin_5), JREGHIGH2.13 (Pin_13)
- new net IN_ACC3: JALU2.2 (Pin_2), JDBG1.6 (Pin_6), JREGHIGH2.14 (Pin_14)
- new net IN_ACC4: JALU2.7 (Pin_7), JDBG1.7 (Pin_7), JREGHIGH2.11 (Pin_11)
- new net IN_ACC5: JALU2.5 (Pin_5), JDBG1.8 (Pin_8), JREGHIGH2.12 (Pin_12)
- new net IN_ACC6: JALU2.3 (Pin_3), JDBG1.9 (Pin_9), JREGHIGH2.9 (Pin_9)
- new net WRITEID0: JALU2.16 (Pin_16), JREGHIGH1.10 (Pin_10), JREGLOW1.10 (Pin_10)
- new net WRITEID1: JALU2.14 (Pin_14), JREGHIGH1.8 (Pin_8), JREGLOW1.8 (Pin_8)
- new net WRITEID2: JALU2.12 (Pin_12), JREGHIGH1.6 (Pin_6), JREGLOW1.6 (Pin_6)
- new net WRITEID3: JALU2.10 (Pin_10), JREGHIGH1.7 (Pin_7), JREGLOW1.9 (Pin_9)
- new net ~{SKIP_ME}: UDEMUX1.6 (G1), UNAND1.1, UREG1.2 (Q0)
- no-connect marks 4 -> 14
Other:
- removed sheet Daughter Boards
- note added: "7 WEN2 9 ~{WEN1} 11 ~{WEN0}"
- note added: "ALUMux"
- note added: "DEBUG"
- note added: "Jump: - Writes MEM to PC"
- note added: "Motherboard TODO: - Reverse-Bias/OVP (How?) - Check memory timing/WE - CheckAllPinout - Skip inst don't carry - Regdata -> OctalBuffer -> MemData"
- note added: "Power"
- note added: "Program Counter"
- note added: "Propogation Delays (Not Counting Transition Times) HCS00 NAND 13ns HC08 AND 14ns HCS14 INV 17ns HCS32 OR 13ns HCS86 XOR 13ns HCS138 DEMUX 19ns HCS151 8:1MUX 14ns, any D HCS153 4:1MUX 17ns, ab input HCS157 2:1MUX 19ns, ab input AC283 ADD 36ns, 2-in-series"
- note added: "RAM"
- note added: "RESET SYSTEM"
- note added: "ROM"
- note added: "Register File High"
- note added: "Register File Low"
- note added: "Skip: Cur Inst: Write ACC to ACC Next inst: Don't change carry register Next inst: Don't change register file Next inst: Don't write to memory"
- note added: "TODO crowbar"
- note added: "~{CS} set low on addr matching AND ~{CLK} (Drive internally) ~{OE} set low on RB instruction (Drive from mobo) ~{WE} set low on WB instruction (Drive from mobo)"
- note added: "~{REN}"
- note removed: "55ns"
- note removed: "COUNTER"
- note removed: "HC86 -> 20ns"
- note removed: "HCS14 = 17ns"
- note removed: "Motherboard Systems: - Opcode decoding - Reverse Bias Protection? - 5V zener diodes? - Check memory timing/WE?"
- note removed: "POWER"
- note removed: "Propogation Delays (Not Counting Transition Times) HCS00 NAND 13ns HC08 AND 14ns HCS14 INV 17ns HCS32 OR 13ns HCS86 XOR 13ns HCS138 DEMUX 19ns HCS151 8:1MUX 14ns, any D HCS153 4:1MUX 17ns, ab input HCS157 2:1MUX 19ns, ab input AC283 ADD 36ns, 2-in-series HCS684 CMP 69ns"
- note removed: "Skip has to do the following to the next instruction: ? Don't change carry register ? Don't change register file ? Don't write to memory"
- note removed: "TODO Replace with APX823-46W5G-7"
- moved on the sheet: C1, C10, C11, C12, C13, C14, C15, C16, C17, C18, C19, C2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

Commit message: Motherboard Layout: Most Traces Done
~30 traces left for motherboard, then it's all ready for ordering!
Parts:
- removed C26, C28: .1uF, Capacitor_SMD:C_1206_3216Metric_Pad1.33x1.80mm_HandSolder, symbol Device:C
- removed F1: Fastblow Fuse, symbol Device:Fuse
- added C29, C30, C31, C32, C33, C34, C35: 10uF, Capacitor_SMD:C_1206_3216Metric_Pad1.33x1.80mm_HandSolder, symbol Device:C
- added D2: DDZ5V6BSF-7, 000custom:SODFL2512X75N, symbol Device:D_Zener
- added F2: 250mA, aFootprint:fuse-0679h, symbol Device:Fuse
- added JREGHIGH2: Conn2x8, Connector_PinSocket_2.54mm:PinSocket_2x08_P2.54mm_Vertical, symbol Connector_Generic:Conn_02x08_Odd_Even
- C27: value .1uF -> 10uF
- TPROM15: footprint (none) -> TestPoint:TestPoint_THTPad_1.5x1.5mm_Drill0.7mm
- U3: value APX823-46W5G-7 -> APX823
- U4: value 74HCS244 -> 74x244
- renumbered JREGHIGH2 to JREGLOW3, JREGLOW2 to JREGLOW4
Connections:
- net GND: now also C29.2, C30.2, C31.2, C32.2, C33.2, C34.2, C35.2, D2.2 (A); no longer JMEM_A2.14 (Pin_14), JMEM_B2.14 (Pin_14), JMEM_C2.14 (Pin_14), JMEM_D2.14 (Pin_14), U2MUX4.14 (I0d), U4.9 (2Y3)
- net IN_ACC0: now also JREGLOW3.7 (Pin_7); no longer JREGLOW3.15 (Pin_15)
- net IN_ACC1: now also JREGLOW3.8 (Pin_8); no longer JREGLOW3.16 (Pin_16)
- net IN_ACC2: now also JREGLOW3.5 (Pin_5); no longer JREGLOW3.13 (Pin_13)
- net IN_ACC3: now also JREGLOW3.6 (Pin_6); no longer JREGLOW3.14 (Pin_14)
- net IN_ACC4: now also JREGLOW3.3 (Pin_3); no longer JREGLOW3.11 (Pin_11)
- net IN_ACC5: now also JREGLOW3.4 (Pin_4); no longer JREGLOW3.12 (Pin_12)
- net IN_ACC6: now also JREGLOW3.1 (Pin_1); no longer JREGLOW3.9 (Pin_9)
- net IN_ACC7: now also JREGLOW3.2 (Pin_2); no longer JREGLOW3.10 (Pin_10)
- net MEM_ADDR0: no longer UR1.3 (D0)
- net MEM_ADDR1: no longer UR1.4 (D1)
- net MEM_ADDR10: no longer UR3.5 (D2)
- net MEM_ADDR11: no longer UR3.6 (D3)
- net MEM_ADDR12: no longer UR4.3 (D0)
- net MEM_ADDR13: no longer UR4.4 (D1)
- net MEM_ADDR14: no longer UR4.5 (D2)
- net MEM_ADDR15: no longer UR4.6 (D3)
- net MEM_ADDR2: no longer UR1.5 (D2)
- net MEM_ADDR3: no longer UR1.6 (D3)
- net MEM_ADDR4: no longer UR2.3 (D0)
- net MEM_ADDR5: no longer UR2.4 (D1)
- net MEM_ADDR6: no longer UR2.5 (D2)
- net MEM_ADDR7: no longer UR2.6 (D3)
- net MEM_ADDR8: no longer UR3.3 (D0)
- net MEM_ADDR9: no longer UR3.4 (D1)
- net RCS0: now also JREGLOW3.15 (Pin_15); no longer JREGLOW3.7 (Pin_7)
- net RCS1: now also JREGLOW3.16 (Pin_16); no longer JREGLOW3.8 (Pin_8)
- net RCS2: now also JREGLOW3.13 (Pin_13); no longer JREGLOW3.5 (Pin_5)
- net RCS3: now also JREGLOW3.14 (Pin_14); no longer JREGLOW3.6 (Pin_6)
- net RCS4: now also JREGLOW3.11 (Pin_11); no longer JREGLOW3.3 (Pin_3)
- net RCS5: now also JREGLOW3.12 (Pin_12); no longer JREGLOW3.4 (Pin_4)
- net RCS6: now also JREGLOW3.9 (Pin_9); no longer JREGLOW3.1 (Pin_1)
- net RCS7: now also JREGLOW3.10 (Pin_10); no longer JREGLOW3.2 (Pin_2)
- net VCC: now also C29.1, C30.1, C31.1, C32.1, C33.1, C34.1, C35.1, D2.1 (K), F2.1
- net ~{CARRY_WE}: now also UNAND1.3; no longer UNOT1.6
- net ~{L}: now also UNOT1.5; no longer UNAND1.2
- net at J1.1: now also F2.2
- net ~{MR_BTN}: now reaches SW1.2, U3.3 (~{MR})
- net OPB_IS_IMM renamed OPCODE0
- new net JMPDST0: JREGHIGH2.7 (Pin_7), UR1.3 (D0)
- new net JMPDST1: JREGHIGH2.8 (Pin_8), UR1.4 (D1)
- new net JMPDST10: JREGHIGH2.13 (Pin_13), UR3.5 (D2)
- new net JMPDST11: JREGHIGH2.14 (Pin_14), UR3.6 (D3)
- new net JMPDST12: JREGHIGH2.11 (Pin_11), UR4.3 (D0)
- new net JMPDST13: JREGHIGH2.12 (Pin_12), UR4.4 (D1)
- new net JMPDST14: JREGHIGH2.9 (Pin_9), UR4.5 (D2)
- new net JMPDST15: JREGHIGH2.10 (Pin_10), UR4.6 (D3)
- new net JMPDST2: JREGHIGH2.5 (Pin_5), UR1.5 (D2)
- new net JMPDST3: JREGHIGH2.6 (Pin_6), UR1.6 (D3)
- new net JMPDST4: JREGHIGH2.3 (Pin_3), UR2.3 (D0)
- new net JMPDST5: JREGHIGH2.4 (Pin_4), UR2.4 (D1)
- new net JMPDST6: JREGHIGH2.1 (Pin_1), UR2.5 (D2)
- new net JMPDST7: JREGHIGH2.2 (Pin_2), UR2.6 (D3)
- new net JMPDST8: JREGHIGH2.15 (Pin_15), UR3.3 (D0)
- new net JMPDST9: JREGHIGH2.16 (Pin_16), UR3.4 (D1)
- new net L: UNAND1.2, UNOT1.6
- new net MEM_DATA7: JMEM_A2.14 (Pin_14), JMEM_B2.14 (Pin_14), JMEM_C2.14 (Pin_14), JMEM_D2.14 (Pin_14), U2MUX4.14 (I0d), U4.9 (2Y3)
Other:
- note added: "<-- Roughly the Reactance"
- note added: "CE2 set on addr matching (Internal Logic) CE# to CLK or nothing (Drive from mobo) ~{OE} set low on RB instruction (Drive from mobo) ~{WE} set low on WB instruction (Drive from mobo) This way, it would drop CS before the data changes"
- note added: "Daughter Decoupling Capacitors"
- note added: "Motherboard Done: - Reverse-Bias/OVP (How?) - Check memory timing/WE - CheckAllPinout - Skip inst don't carry - Regdata -> OctalBuffer -> MemData - Consider JMP mem reg being different than WB/RB register"
- note added: "OPB_IS_IMM ->"
- note added: "OPCODE1 = IN_R1"
- note added: "Skip: Cur Inst: Don't write mem/reg Next inst: Don't change carry register Next inst: Don't change register file Next inst: Don't write to memory Next inst: Don't skip or jump"
- note removed: "<-- Roughly the Reactance?"
- note removed: "Motherboard TODO: - Reverse-Bias/OVP (How?) - Check memory timing/WE - CheckAllPinout - Skip inst don't carry - Regdata -> OctalBuffer -> MemData"
- note removed: "Skip: Cur Inst: Write ACC to ACC Next inst: Don't change carry register Next inst: Don't change register file Next inst: Don't write to memory"
- note removed: "TODO crowbar"
- note removed: "~{CS} set low on addr matching AND ~{CLK} (Drive internally) ~{OE} set low on RB instruction (Drive from mobo) ~{WE} set low on WB instruction (Drive from mobo)"
- moved on the sheet: C1, C10, C11, C12, C13, C14, C15, C16, C17, C18, C19, C2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

Commit message: Motherboard V1
Parts:
- J1: footprint Connector_BarrelJack:BarrelJack_Horizontal -> 000custom:BarrelJack_Horizontal
Connections:
- net CLK_INT: now reaches JP1.1 (A), UNOT1.2
Changed lines of the file:
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@@
     (effects (font (size 1.27 1.27)) (justify right bottom))
+  )
+  (label "CLK_INT" (at 83.82 176.53 0) (fields_autoplaced)
+    (effects (font (size 1.27 1.27)) (justify left bottom))
   )
   (label "CARRY" (at 101.6 266.7 180) (fields_autoplaced)
@@
       (effects (font (size 1.27 1.27)))
     )
-    (property "Footprint" "Connector_BarrelJack:BarrelJack_Horizontal" (at 26.67 103.886 0)
-      (effects (font (size 1.27 1.27)) hide)
-    )
+    (property "Footprint" "000custom:BarrelJack_Horizontal" (at 26.67 103.886 0)
+      (effects (font (size 1.27 1.27)) hide)
+    )
